File: PCB/Hackpad.kicad_pcb (KiCad board)
At the start: 2 copper layers, 62 x 89 mm, 21 parts, among them J1 OLED_128x64, SW1 RotaryEncoder_Switch, U1 MCU_Seeed_XIAO_RP2040

Commit message: Updated Image Files v3
Connections:
- SW1 pad C: 3.3V -> GROUND
Changed lines of the file:
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@@
 			(sketchdnponfab yes)
 			(crossoutdnponfab yes)
-			(subtractmaskfromsilk no)
+			(subtractmaskfromsilk yes)
 			(outputformat 1)
 			(mirror no)
-			(drillshape 1)
+			(drillshape 0)
 			(scaleselection 1)
-			(outputdirectory "")
+			(outputdirectory "../../Downloads/")
 		)
 	)
@@
 			(layers "*.Cu" "*.Mask")
 			(remove_unused_layers no)
-			(net 23 "3.3V")
+			(net 17 "GROUND")
 			(pinfunction "C")
 			(pintype "passive")
